File: CurrentSens.kicad_sch (KiCad schematic)
At the start: 25 parts, among them J1 USB_C_Receptacle_USB2.0, J102 Conn_01x01, J104 Conn_01x01, J105 Conn_Coaxial, J106 Conn_01x04

Commit message: Some fixes for first production run at aisler - change inductor - add 3D data - fix references in silkscreen
Parts:
- L101: footprint Inductor_SMD:L_Ferrocore_DLG-0403 -> CurrentSens:SDR0604330KL
Changed lines of the file:
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@@
       (effects (font (size 1.27 1.27)))
     )
-    (property "Footprint" "Inductor_SMD:L_Ferrocore_DLG-0403" (at 122.555 30.48 0)
+    (property "Footprint" "CurrentSens:SDR0604330KL" (at 122.555 30.48 0)
       (effects (font (size 1.27 1.27)) hide)
     )
